File: circuit/PicoThermoClock.kicad_pcb (KiCad board)
At the start: 2 copper layers, 100 x 100 mm, 41 parts, among them J1 USB_B_Micro, J2 AVR-ISP-6, J3 Conn_01x03, J4 Conn_01x03, Q1 SS9012H, Q2 SS9012H, Q3 SS9012H, Q4 SS9012H, Q5 C1815GR, SW1 SW_Push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

Commit message: PRO: import JLCPCB rules from below github project
https://github.com/sethhillbrand/kicad_templates
Other:
- copper layers 2 -> 4
- net class Default: clearance 0.3 -> 0.127; trace_width 0.25 -> 0.127; via_dia 0.8 -> 0.6; via_drill 0.4 -> 0.3
- rule trace_clearance: 0.3 -> 0.127
- rule trace_min: 0.25 -> 0.127
- rule via_min_size: 0.4 -> 0.6

Commit message: PCB: fix missing GND pin connection
Routing:
- net GND: track 0.00 -> 2.44 mm
